Commit message: moveit enabled

File: braccio_support/urdf/braccio.urdf (robot description, URDF)
Before this commit: robot braccio_arm, 4 links, 2 joints
Links:
- removed link braccio_base_link
- removed link braccio_tool0
- added link base_link
- added link braccio_ee
- added link braccio_link_2; collision mesh filename=package://braccio_support/meshes/collision/arm_m23.stl; visual mesh filename=package://braccio_support/meshes/visual/arm_m23.stl
- added link braccio_link_3; collision mesh filename=package://braccio_support/meshes/collision/arm_m23.stl; visual mesh filename=package://braccio_support/meshes/visual/arm_m23.stl
- added link braccio_link_4; collision mesh filename=package://braccio_support/meshes/collision/hand.stl; visual mesh filename=package://braccio_support/meshes/visual/hand.stl
- added link braccio_link_5; collision mesh filename=package://braccio_support/meshes/collision/gripper.stl; visual mesh filename=package://braccio_support/meshes/visual/gripper.stl
- link braccio_base: geometry collision mesh filename=package://braccio_support/meshes/collision/base_plate.stl; visual mesh filename=package://braccio_support/meshes/visual/base_plate.stl
- link braccio_link_1: geometry collision mesh filename=package://braccio_support/meshes/collision/base_m1.stl; visual mesh filename=package://braccio_support/meshes/visual/base_m1.stl
Joints:
- added joint braccio_joint_2: type revolute, parent braccio_link_1, child braccio_link_2, origin xyz=0 0 0 rpy=0 -1.570796327 0, axis 0 0 1, limit lower=-3.14 upper=3.14 effort=0 velocity=3.67
- added joint braccio_joint_3: type revolute, parent braccio_link_2, child braccio_link_3, origin xyz=12.5 0 0 rpy=0 0 0, axis 0 0 1, limit lower=-3.14 upper=3.14 effort=0 velocity=3.67
- added joint braccio_joint_4: type revolute, parent braccio_link_3, child braccio_link_4, origin xyz=12.5 0 0 rpy=0 0 0, axis 0 0 1, limit lower=-3.14 upper=3.14 effort=0 velocity=3.67
- added joint braccio_joint_5: type revolute, parent braccio_link_4, child braccio_link_5, origin xyz=6.1 0 0 rpy=0 1.570796327 0, axis 0 0 1, limit lower=-3.14 upper=3.14 effort=0 velocity=3.67
- added joint braccio_joint_ee: type fixed, parent braccio_link_5, child braccio_ee, origin xyz=0 0.45 12.6 rpy=0 0 0
- joint braccio_base_link-base: origin xyz=0 0 0.0 rpy=0 0 0 -> xyz=0 0 0 rpy=0 0 0
- joint braccio_joint_1: origin xyz=0 0 0.004 rpy=0 0 0 -> xyz=0 0 7.22 rpy=0 0 0; parent braccio_base_link -> braccio_base

Commit message: Driver seems to be working -- more tests needed

File: braccio_support/urdf/braccio.urdf (robot description, URDF)
Before this commit: robot braccio_arm, 8 links, 7 joints
Joints:
- joint braccio_joint_1: limit lower=-3.14 upper=3.14 effort=0 velocity=3.67 -> lower=0 upper=3.14 effort=0 velocity=3.67
- joint braccio_joint_2: limit lower=-3.14 upper=3.14 effort=0 velocity=3.67 -> lower=0.26 upper=2.88 effort=0 velocity=3.67
- joint braccio_joint_3: limit lower=-3.14 upper=3.14 effort=0 velocity=3.67 -> lower=0 upper=3.14 effort=0 velocity=3.67
- joint braccio_joint_4: limit lower=-3.14 upper=3.14 effort=0 velocity=3.67 -> lower=0 upper=3.14 effort=0 velocity=3.67
- joint braccio_joint_5: limit lower=-3.14 upper=3.14 effort=0 velocity=3.67 -> lower=0 upper=3.14 effort=0 velocity=3.67

Commit message: Trying to get the Action Server to work

File: braccio_support/urdf/braccio.urdf (robot description, URDF)
Before this commit: robot braccio_arm, 8 links, 7 joints
Joints:
- joint braccio_joint_1: limit lower=0 upper=3.14 effort=0 velocity=3.67 -> lower=-1.57 upper=1.57 effort=0 velocity=3.67
- joint braccio_joint_2: limit lower=0.26 upper=2.88 effort=0 velocity=3.67 -> lower=-1.31 upper=1.31 effort=0 velocity=3.67
- joint braccio_joint_3: limit lower=0 upper=3.14 effort=0 velocity=3.67 -> lower=-1.57 upper=1.57 effort=0 velocity=3.67
- joint braccio_joint_4: limit lower=0 upper=3.14 effort=0 velocity=3.67 -> lower=-1.57 upper=1.57 effort=0 velocity=3.67
- joint braccio_joint_5: limit lower=0 upper=3.14 effort=0 velocity=3.67 -> lower=-1.57 upper=1.57 effort=0 velocity=3.67

File: braccio_support/urdf/braccio_macro.xacro (robot description, xacro)
@@ -109,5 +109,5 @@
       <child link="${prefix}_link_1"/>
       <axis xyz="0 0 1"/>
-      <limit lower="0" upper="3.14" effort="0" velocity="3.67"/>
+      <limit lower="-1.57" upper="1.57" effort="0" velocity="3.67"/>
     </joint>
     <joint name="${prefix}_joint_2" type="revolute">
@@ -116,5 +116,5 @@
       <child link="${prefix}_link_2"/>
       <axis xyz="0 0 1"/>
-      <limit lower="0.26" upper="2.88" effort="0" velocity="3.67"/>
+      <limit lower="-1.31" upper="1.31" effort="0" velocity="3.67"/>
     </joint>
     <joint name="${prefix}_joint_3" type="revolute">
@@ -123,5 +123,5 @@
       <child link="${prefix}_link_3"/>
       <axis xyz="0 0 1"/>
-      <limit lower="0" upper="3.14" effort="0" velocity="3.67"/>
+      <limit lower="-1.57" upper="1.57" effort="0" velocity="3.67"/>
     </joint>
     <joint name="${prefix}_joint_4" type="revolute">
@@ -130,5 +130,5 @@
       <child link="${prefix}_link_4"/>
       <axis xyz="0 0 1"/>
-      <limit lower="0" upper="3.14" effort="0" velocity="3.67"/>
+      <limit lower="-1.57" upper="1.57" effort="0" velocity="3.67"/>
     </joint>
     <joint name="${prefix}_joint_5" type="revolute">
@@ -137,5 +137,5 @@
       <child link="${prefix}_link_5"/>
       <axis xyz="0 0 1"/>
-      <limit lower="0" upper="3.14" effort="0" velocity="3.67"/>
+      <limit lower="-1.57" upper="1.57" effort="0" velocity="3.67"/>
     </joint>
     <joint name="${prefix}_joint_ee" type="fixed">

Commit message: Braccio follows the trajectory in RViz

File: braccio_support/urdf/braccio.urdf (robot description, URDF)
Before this commit: robot braccio_arm, 8 links, 7 joints
Joints:
- joint braccio_joint_1: axis 0 0 1 -> 0 0 -1
- joint braccio_joint_5: axis 0 0 1 -> 0 0 -1

File: braccio_support/urdf/braccio_macro.xacro (robot description, xacro)
@@ -108,5 +108,5 @@
       <parent link="${prefix}_base"/>
       <child link="${prefix}_link_1"/>
-      <axis xyz="0 0 1"/>
+      <axis xyz="0 0 -1"/>
       <limit lower="-1.57" upper="1.57" effort="0" velocity="3.67"/>
     </joint>
@@ -136,5 +136,5 @@
       <parent link="${prefix}_link_4"/>
       <child link="${prefix}_link_5"/>
-      <axis xyz="0 0 1"/>
+      <axis xyz="0 0 -1"/>
       <limit lower="-1.57" upper="1.57" effort="0" velocity="3.67"/>
     </joint>
